Commit message: update deploy code, add sim2sim README, cleanup probe scripts
- Deploy: fix joint name matching (joint1-a1_r), add acceleration
  compensation in phase correction, add obs/action CSV logging,
  add ball observation columns to deploy CSV
- Add sim2sim & deploy README with known issues and TODO
- Remove obsolete probe/diagnostic scripts (v56-v85, fk_probe, etc.)
- Update env_cfg, play.py, sim2sim scripts, deploy header

Co-Authored-By: Claude Opus 4.6 <noreply@anthropic.com>

File: x1/x1/urdf/x1.urdf (robot description, URDF)
Before this commit: robot X1, 22 links, 21 joints
Joints:
- joint joint_yb_2: axis 0 0 1 -> 0 0 -1; limit lower=-3.081 upper=0.314 effort=0 velocity=0 -> lower=-0.314 upper=3.081 effort=0 velocity=0
